Commit message: Added stl import code, but stl not well formatted.

File: jaws2_description/urdf/jaws2_housing.urdf.xacro (robot description, xacro)
@@ -48,4 +48,5 @@
       <geometry>
         <sphere radius="${housing_radius}" />
+        <!-- <mesh filename="package://jaws2_description/meshes/dome.stl" /> -->
       </geometry>
       <material name="Grey" />
