Commit message: Updated description to add controls.

File: jaws2_description/urdf/jaws2.gazebo.xacro (robot description, xacro)
@@ -1,15 +1,12 @@
 <?xml version="1.0"?>
 <robot xmlns:xacro="http://ros.org/wiki/xacro">
-<!--  Gazebo  -->
   <gazebo>
     <!--  Buoyancy  -->
     <plugin name="BuoyancyPlugin" filename="libBuoyancyPlugin.so" />
-<!--
-          <link name="dome">
-            <center_of_volume>${dome_volume_ctr}</center_of_volume>
-            <volume>${dome_volume}</volume>
-          </link>
--->
-    <!--  Controls  -->
+    <!--  Servo Simulation Interface  -->
+    <plugin name="gazebo_ros_control" filename="libgazebo_ros_control.so">
+      <robotNamespace>/jaws2</robotNamespace>
+    </plugin>
+    <!--  Thruster Simulation Interface  -->
     <plugin filename="libgazebo_ros_force.so" name="gazebo_ros_force">
       <bodyName>aft_thruster</bodyName>
@@ -25,5 +22,5 @@
     </plugin>
   </gazebo>
-  <!--  Simulation Materials  -->
+  <!--  Gazebo Materials  -->
   <gazebo reference="dome">
     <material>Gazebo/Grey</material>

File: jaws2_description/urdf/jaws2.urdf (robot description, URDF)
Before this commit: robot jaws2, 23 links, 22 joints
Links:
- added link housing, mass 1.8914
- link base_link: mass 5.7914 -> None
Joints:
- added joint housing: type fixed, parent base_link, child housing
- joint aft_gasket_joint: parent base_link -> housing
- joint aft_thruster_mount_joint: parent base_link -> housing
- joint aft_thruster_riser_joint: parent base_link -> housing
- joint fwd_gasket_joint: parent base_link -> housing
- joint mid_housing_joint: parent base_link -> housing
- joint port_servo: parent base_link -> housing
- joint port_thruster_mount_joint: parent base_link -> housing
- joint stbd_servo: parent base_link -> housing
- joint stbd_thruster_mount_joint: parent base_link -> housing

File: jaws2_description/urdf/jaws2.urdf.xacro (robot description, xacro)
@@ -1,7 +1,34 @@
 <?xml version="1.0"?>
 <robot name="jaws2" xmlns:xacro="http://ros.org/wiki/xacro">
+  <!-- Servo Interface -->
+  <transmission name="port">
+    <type>transmission_interface/SimpleTransmission</type>
+    <joint name="port_servo">
+      <hardwareInterface>EffortJointInterface</hardwareInterface>
+    </joint>
+    <actuator name="port_servo_motor">
+      <hardwareInterface>EffortJointInterface</hardwareInterface>
+      <mechanicalReduction>1</mechanicalReduction>
+    </actuator>
+  </transmission>
+  <transmission name="stbd">
+    <type>transmission_interface/SimpleTransmission</type>
+    <joint name="stbd_servo">
+      <hardwareInterface>EffortJointInterface</hardwareInterface>
+    </joint>
+    <actuator name="stbd_servo_motor">
+      <hardwareInterface>EffortJointInterface</hardwareInterface>
+      <mechanicalReduction>1</mechanicalReduction>
+    </actuator>
+  </transmission>
+  <!--  Dummy Link  -->
+  <link name="base_link" />
+  <joint name="housing" type="fixed">
+    <parent link="base_link" />
+    <child link="housing" />
+  </joint>
+  <xacro:include filename="jaws2_housing.urdf.xacro" />
+  <xacro:include filename="jaws2_mounting.urdf.xacro" />
   <xacro:include filename="jaws2_properties.urdf.xacro" />
-  <xacro:include filename="jaws2_housing.urdf.xacro" />
-  <xacro:include filename="jaws2_visual.urdf.xacro" />
   <xacro:include filename="jaws2.gazebo.xacro" />
   <xacro:include filename="seabotix_thrusters.urdf.xacro" />

File: jaws2_description/urdf/jaws2_housing.urdf.xacro (robot description, xacro)
@@ -1,5 +1,6 @@
 <?xml version="1.0"?>
 <robot xmlns:xacro="http://ros.org/wiki/xacro">
-  <link name="base_link">
+  <!--  Main Housing Inertia  -->
+  <link name="housing">
     <inertial>
       <mass value="${housing_mass}" />
@@ -7,11 +8,43 @@
     </inertial>
   </link>
-    <xacro:macro name="gasket" params="pre lnk fa d">
-    <joint name="${pre}_gasket_joint" type="fixed">
-      <origin xyz="${fa*gasket_x} 0 0" rpy="0 0 0" />
-      <parent link="base_link" />
-      <child link="${pre}_gasket" />
+  <!--  Main Housing Volume  -->
+  <xacro:macro name="joints" params="prefix d p">
+    <joint name="${prefix}_housing_joint" type="fixed">
+      <origin xyz="${d} 0 0" rpy="0 0 0" />
+      <parent link="${p}" />
+      <child link="${prefix}_housing" />
     </joint>
-    <link name="${pre}_gasket">
+  </xacro:macro>
+  <xacro:joints prefix="fwd" d="${(fwd_length+mid_length)/2}" p="mid_housing" />
+  <xacro:joints prefix="mid" d="${(aft_length-fwd_length)/2}" p="housing" />
+  <xacro:joints prefix="aft" d="${-(aft_length+mid_length)/2}" p="mid_housing" />
+  <xacro:macro name="links" params="prefix radius length">
+    <link name="${prefix}_housing">
+      <visual>
+        <xacro:insert_block name="cylinder_fix" />
+        <geometry>
+          <cylinder radius="${radius}" length="${length}" />
+        </geometry>
+        <material name="FlatBlack" />
+      </visual>
+      <collision>
+        <xacro:insert_block name="cylinder_fix" />
+        <geometry>
+          <cylinder radius="${radius}" length="${length}" />
+        </geometry>
+      </collision>
+    </link>
+  </xacro:macro>
+  <xacro:links prefix="fwd" radius="${housing_radius}" length="${fwd_length}"/>
+  <xacro:links prefix="mid" radius="${middle_radius}" length="${mid_length}"/>
+  <xacro:links prefix="aft" radius="${housing_radius}" length="${aft_length}"/>
+  <!--  Gaskets  -->
+  <xacro:macro name="gasket" params="prefix reflect">
+    <joint name="${prefix}_gasket_joint" type="fixed">
+      <origin xyz="${reflect*gasket_x} 0 0" rpy="0 0 0" />
+      <parent link="housing" />
+      <child link="${prefix}_gasket" />
+    </joint>
+    <link name="${prefix}_gasket">
       <inertial>
         <mass value="${gasket_mass}" />
@@ -32,12 +65,18 @@
       </collision>
     </link>
-    <joint name="${lnk}_joint" type="fixed">
-      <origin xyz="${d} 0 0" rpy="0 0 0" />
-      <parent link="${pre}_gasket" />
-      <child link="${lnk}" />
-    </joint>
   </xacro:macro>
-  <xacro:gasket pre="fwd" lnk="dome" fa="1" d="${gasket_length/2}" />
-  <xacro:gasket pre="aft" lnk="endcap" fa="-1" d="${-(endcap_length+gasket_length)/2}" />
+  <xacro:gasket prefix="fwd" reflect="1" />
+  <xacro:gasket prefix="aft" reflect="-1" />
+  <!--  Dome/Endcap  -->
+  <joint name="dome_joint" type="fixed">
+    <origin xyz="${gasket_length/2} 0 0" rpy="0 0 0" />
+    <parent link="fwd_gasket" />
+    <child link="dome" />
+  </joint>
+  <joint name="endcap_joint" type="fixed">
+    <origin xyz="${-(endcap_length+gasket_length)/2} 0 0" rpy="0 0 0" />
+    <parent link="aft_gasket" />
+    <child link="endcap" />
+  </joint>
   <link name="dome">
     <inertial>
@@ -77,55 +116,3 @@
     </collision>
   </link>
-  <xacro:macro name="servo" params="prefix reflect mirror">
-    <joint name="${prefix}_servo" type="revolute">
-      <origin xyz="${shaft_x} ${reflect*shaft_y} 0" rpy="0 ${-M_PI/2} ${mirror}"/>
-      <parent link="base_link" />
-      <child link="${prefix}_servo_shaft" />
-      <axis xyz="0 1 0" />
-      <limit lower="${-2*M_PI/3}" upper="${2*M_PI/3}" effort="1.4994" velocity="1.9666" />
-    </joint>
-    <link name="${prefix}_servo_shaft">
-      <inertial>
-        <mass value="${shaft_mass}" />
-        <xacro:insert_block name="shaft_inertia" />
-      </inertial>
-      <visual>
-        <origin xyz="0 0 0" rpy="${M_PI/2} 0 0" />
-        <geometry>
-          <cylinder radius="${shaft_radius}" length="${shaft_length}" />
-        </geometry>
-        <material name="DarkGrey" />
-      </visual>
-      <collision>
-        <origin xyz="0 0 0" rpy="${M_PI/2} 0 0" />
-        <geometry>
-          <cylinder radius="${shaft_radius}" length="${shaft_length}" />
-        </geometry>
-      </collision>
-    </link>
-  </xacro:macro>
-  <xacro:servo prefix="port" reflect="1" mirror="0"/>
-  <xacro:servo prefix="stbd" reflect="-1" mirror="${M_PI}"/>
-  <link name="aft_thruster_riser">
-    <inertial>
-      <mass value="${riser_mass}" />
-      <xacro:insert_block name="riser_inertia" />
-    </inertial>
-    <visual>
-      <geometry>
-        <box size="${0.75*riser_length} ${0.55*riser_width} ${riser_height}" />
-      </geometry>
-      <material name="DarkGrey" />
-    </visual>
-    <collision>
-      <geometry>
-        <box size="${riser_length} ${riser_width} ${riser_height}" />
-      </geometry>
-    </collision>
-  </link>
-  <joint name="aft_thruster_riser_joint" type="fixed">
-    <origin xyz="${riser_x} 0 ${riser_z}" rpy="0 0 0" />
-    <parent link="base_link" />
-    <child link="aft_thruster_riser" />
-  </joint>
 </robot>

File: jaws2_description/urdf/jaws2_properties.urdf.xacro (robot description, xacro)
@@ -2,5 +2,41 @@
 <robot xmlns:xacro="http://ros.org/wiki/xacro">
   <xacro:property name="M_PI" value="3.14159266" />
-<!-- Port & Stbd Thruster Servo Shafts -->
+  <!--  Housing Properties  -->
+  <xacro:property name="housing_radius" value="0.0762" />
+  <xacro:property name="middle_radius" value="0.06985" />
+  <xacro:property name="fwd_length" value="0.0492" />
+  <xacro:property name="mid_length" value="0.2826" />
+  <xacro:property name="aft_length" value="0.0238" />
+  <xacro:property name="housing_mass" value="1.8914" />
+  <xacro:property name="housing_inertia">
+    <inertia ixx="0.00921641" ixy="0.0" ixz="0.0"
+             iyy="0.03285281" iyz="0.0"
+             izz="0.03285281" />
+  </xacro:property>
+  <!-- Gasket Properties  -->
+  <xacro:property name="gasket_length" value="0.0032" />
+  <xacro:property name="gasket_x" value="0.1794" />
+  <xacro:property name="gasket_mass" value="0.0165" />
+  <xacro:property name="gasket_inertia">
+    <inertia ixx="0.00004790" ixy="0.0" ixz="0.0"
+             iyy="0.00002397" iyz="0.0"
+             izz="0.00002397" />
+  </xacro:property>
+  <!--  Dome Properties  -->
+  <xacro:property name="dome_mass" value="0.7700" />
+  <xacro:property name="dome_inertia">
+    <inertia ixx="0.003" ixy="0.0" ixz="0.0"
+             iyy="0.003" iyz="0.0"
+             izz="0.003" />
+  </xacro:property>
+  <!--  Endcap Properties  -->
+  <xacro:property name="endcap_length" value="0.0200" />
+  <xacro:property name="endcap_mass" value="0.1925" />
+  <xacro:property name="endcap_inertia">
+  <inertia ixx="0.000" ixy="0.0" ixz="0.0"
+           iyy="0.003" iyz="0.0"
+           izz="0.003" />
+  </xacro:property>
+<!--  Port & Stbd Servo Propeties  -->
   <xacro:property name="shaft_radius" value="0.01580619" />
   <xacro:property name="shaft_length" value="0.02381250" />
@@ -13,5 +49,5 @@
              izz="0.00000444" />
   </xacro:property>
-<!-- Aft Thruster Riser -->
+<!--  Aft Thruster Riser Properties  -->
   <xacro:property name="riser_length" value="0.0260" />
   <xacro:property name="riser_width" value="0.0260" />
@@ -25,40 +61,23 @@
              izz="0.00000262" />
   </xacro:property>
-<!-- Housing -->
-  <xacro:property name="housing_radius" value="0.0762" />
-  <xacro:property name="middle_radius" value="0.06985" />
-  <xacro:property name="fwd_length" value="0.0492" />
-  <xacro:property name="mid_length" value="0.2826" />
-  <xacro:property name="aft_length" value="0.0238" />
-  <xacro:property name="housing_mass" value="5.7914" />
-  <!-- Mass: 1.8914 -->
-  <xacro:property name="housing_inertia">
-    <inertia ixx="0.00921641" ixy="0.0" ixz="0.0"
-             iyy="0.03285281" iyz="0.0"
-             izz="0.03285281" />
-  </xacro:property>
-  <xacro:property name="gasket_length" value="0.0032" />
-  <xacro:property name="gasket_x" value="0.1794" />
-  <xacro:property name="gasket_mass" value="0.0165" />
-  <xacro:property name="gasket_inertia">
-    <inertia ixx="0.00004790" ixy="0.0" ixz="0.0"
-             iyy="0.00002397" iyz="0.0"
-             izz="0.00002397" />
-  </xacro:property>
-  <xacro:property name="dome_mass" value="0.7700" />
-  <xacro:property name="dome_inertia">
-    <inertia ixx="0.003" ixy="0.0" ixz="0.0"
-             iyy="0.003" iyz="0.0"
-             izz="0.003" />
-  </xacro:property>
-  <xacro:property name="endcap_length" value="0.0200" />
-  <xacro:property name="endcap_mass" value="0.1925" />
-  <xacro:property name="endcap_inertia">
-  <inertia ixx="0.000" ixy="0.0" ixz="0.0"
-           iyy="0.003" iyz="0.0"
-           izz="0.003" />
-  </xacro:property>
+  <!--  Miscellaneous  -->
   <xacro:property name="cylinder_fix">
     <origin xyz="0 0 0" rpy="0 ${M_PI/2} 0" />
   </xacro:property>
+    <!--  Rviz Materials  -->
+    <material name="FlatBlack">
+      <color rgba="0.1 0.1 0.1 1.0" />
+    </material>
+    <material name="DarkGrey">
+      <color rgba="0.175 0.175 0.175 1.0" />
+    </material>
+    <material name="Grey">
+      <color rgba="0.3 0.3 0.3 1.0" />
+    </material>
+    <material name="GreyTransparent">
+      <color rgba="0.5 0.5 0.5 0.5" />
+    </material>
+    <material name="Orange">
+      <color rgba="1 0.5088 0.0468 1" />
+    </material>
 </robot>
