Commit message: The great xacro overhault.

File: jaws2_description/urdf/jaws2.gazebo.xacro (robot description, xacro)
@@ -1,9 +1,12 @@
 <?xml version="1.0"?>
 <robot xmlns:xacro="http://ros.org/wiki/xacro">
+  <!--                                -->
+  <!--  Gazebo Simulation Properties  -->
+  <!--                                -->
   <gazebo>
     <!--  Buoyancy  -->
-    <plugin name="BuoyancyPlugin" filename="libBuoyancyPlugin.so" />
+    <plugin name="BuoyancyPlugin" filename="libBuoyancyPlugin.so"/>
     <!--  Servo Simulation Interface  -->
-    <plugin name="gazebo_ros_control" filename="libgazebo_ros_control.so" />
+    <plugin name="gazebo_ros_control" filename="libgazebo_ros_control.so"/>
     <!--  Thruster Simulation Interface  -->
     <plugin filename="libgazebo_ros_force.so" name="gazebo_ros_force">
@@ -20,5 +23,5 @@
     </plugin>
   </gazebo>
-  <!--  Gazebo Materials  -->
+  <!--  Housing Materials  -->
   <gazebo reference="dome">
     <material>Gazebo/Grey</material>
@@ -50,5 +53,5 @@
     </gazebo>
   </xacro:macro>
-  <xacro:gazebo_materials fa="fwd" ps="port" />
-  <xacro:gazebo_materials fa="aft" ps="stbd" />
+  <xacro:gazebo_materials fa="fwd" ps="port"/>
+  <xacro:gazebo_materials fa="aft" ps="stbd"/>
 </robot>

File: jaws2_description/urdf/jaws2.urdf (robot description, URDF)
Before this commit: robot jaws2, 24 links, 23 joints
Joints:
- joint port_servo: limit lower=-2.09439510667 upper=2.09439510667 effort=1.4994 velocity=1.9666 -> lower=-2.61799388333 upper=2.61799388333 effort=1.4994 velocity=1.96666666
- joint stbd_servo: limit lower=-2.09439510667 upper=2.09439510667 effort=1.4994 velocity=1.9666 -> lower=-2.61799388333 upper=2.61799388333 effort=1.4994 velocity=1.96666666

File: jaws2_description/urdf/jaws2.urdf.xacro (robot description, xacro)
@@ -1,35 +1,31 @@
 <?xml version="1.0"?>
+<!--                                  -->
+<!--  Description of the Jaws 2 ROV.  -->
+<!--                                  -->
+<!--  The Underwater Robotics Team    -->
+<!--     @ The Ohio State University  -->
+<!--                                  -->
 <robot name="jaws2" xmlns:xacro="http://ros.org/wiki/xacro">
-  <!-- Servo Interface -->
-  <transmission name="port">
+<!--                     -->
+<!--  Servo Controllers  -->
+<!--                     -->
+  <xacro:macro name="servo_control" params="prefix">
+  <transmission name="${prefix}">
     <type>transmission_interface/SimpleTransmission</type>
-    <joint name="port_servo">
+    <joint name="${prefix}_servo">
       <hardwareInterface>EffortJointInterface</hardwareInterface>
     </joint>
-    <actuator name="port_servo_motor">
+    <actuator name="${prefix}_servo_motor">
       <hardwareInterface>EffortJointInterface</hardwareInterface>
       <mechanicalReduction>1</mechanicalReduction>
     </actuator>
   </transmission>
-  <transmission name="stbd">
-    <type>transmission_interface/SimpleTransmission</type>
-    <joint name="stbd_servo">
-      <hardwareInterface>EffortJointInterface</hardwareInterface>
-    </joint>
-    <actuator name="stbd_servo_motor">
-      <hardwareInterface>EffortJointInterface</hardwareInterface>
-      <mechanicalReduction>1</mechanicalReduction>
-    </actuator>
-  </transmission>
-  <!--  Dummy Link  -->
-  <link name="base_link" />
-  <joint name="housing" type="fixed">
-    <parent link="base_link" />
-    <child link="housing" />
-  </joint>
-  <xacro:include filename="jaws2_housing.urdf.xacro" />
-  <xacro:include filename="jaws2_mounting.urdf.xacro" />
-  <xacro:include filename="jaws2_properties.urdf.xacro" />
-  <xacro:include filename="jaws2.gazebo.xacro" />
-  <xacro:include filename="seabotix_thrusters.urdf.xacro" />
+  </xacro:macro>
+  <xacro:servo_control prefix="port"/>
+  <xacro:servo_control prefix="stbd"/>
+  <xacro:include filename="jaws2_housing.urdf.xacro"/>
+  <xacro:include filename="jaws2_mounting.urdf.xacro"/>
+  <xacro:include filename="jaws2_properties.urdf.xacro"/>
+  <xacro:include filename="jaws2.gazebo.xacro"/>
+  <xacro:include filename="seabotix_thrusters.urdf.xacro"/>
 </robot>

File: jaws2_description/urdf/jaws2_housing.urdf.xacro (robot description, xacro)
@@ -1,35 +1,44 @@
 <?xml version="1.0"?>
 <robot xmlns:xacro="http://ros.org/wiki/xacro">
-  <!--  Main Housing Inertia  -->
+<!--                      -->
+<!--  Watertight Housing  -->
+<!--                      -->
+  <!--    Required Dummy Link    -->
+  <link name="base_link"/>
+  <!--    Main Housing Inertia    -->
+  <joint name="housing" type="fixed">
+    <parent link="base_link"/>
+    <child link="housing"/>
+  </joint>
   <link name="housing">
     <inertial>
-      <mass value="${housing_mass}" />
-      <xacro:insert_block name="housing_inertia" />
+      <mass value="${housing_mass}"/>
+      <xacro:insert_block name="housing_inertia"/>
     </inertial>
   </link>
-  <!--  Main Housing Volume  -->
+  <!--    Main Housing Volume    -->
   <xacro:macro name="joints" params="prefix d p">
     <joint name="${prefix}_housing_joint" type="fixed">
-      <origin xyz="${d} 0 0" rpy="0 0 0" />
-      <parent link="${p}" />
-      <child link="${prefix}_housing" />
+      <origin xyz="${d} 0 0" rpy="0 0 0"/>
+      <parent link="${p}"/>
+      <child link="${prefix}_housing"/>
     </joint>
   </xacro:macro>
-  <xacro:joints prefix="fwd" d="${(fwd_length+mid_length)/2}" p="mid_housing" />
-  <xacro:joints prefix="mid" d="${(aft_length-fwd_length)/2}" p="housing" />
-  <xacro:joints prefix="aft" d="${-(aft_length+mid_length)/2}" p="mid_housing" />
+  <xacro:joints prefix="fwd" d="${(fwd_length+mid_length)/2}" p="mid_housing"/>
+  <xacro:joints prefix="mid" d="${(aft_length-fwd_length)/2}" p="housing"/>
+  <xacro:joints prefix="aft" d="${-(aft_length+mid_length)/2}" p="mid_housing"/>
   <xacro:macro name="links" params="prefix radius length">
     <link name="${prefix}_housing">
       <visual>
-        <xacro:insert_block name="cylinder_fix" />
+        <xacro:insert_block name="pitch_fix"/>
         <geometry>
-          <cylinder radius="${radius}" length="${length}" />
+          <cylinder radius="${radius}" length="${length}"/>
         </geometry>
-        <material name="FlatBlack" />
+        <material name="FlatBlack"/>
       </visual>
       <collision>
-        <xacro:insert_block name="cylinder_fix" />
+        <xacro:insert_block name="pitch_fix"/>
         <geometry>
-          <cylinder radius="${radius}" length="${length}" />
+          <cylinder radius="${radius}" length="${length}"/>
         </geometry>
       </collision>
@@ -39,78 +48,79 @@
   <xacro:links prefix="mid" radius="${middle_radius}" length="${mid_length}"/>
   <xacro:links prefix="aft" radius="${housing_radius}" length="${aft_length}"/>
-  <!--  Gaskets  -->
+  <!--    Gaskets    -->
   <xacro:macro name="gasket" params="prefix reflect">
     <joint name="${prefix}_gasket_joint" type="fixed">
-      <origin xyz="${reflect*gasket_x} 0 0" rpy="0 0 0" />
-      <parent link="housing" />
-      <child link="${prefix}_gasket" />
+      <origin xyz="${reflect*gasket_x} 0 0" rpy="0 0 0"/>
+      <parent link="housing"/>
+      <child link="${prefix}_gasket"/>
     </joint>
     <link name="${prefix}_gasket">
       <inertial>
-        <mass value="${gasket_mass}" />
-        <xacro:insert_block name="gasket_inertia" />
+        <mass value="${gasket_mass}"/>
+        <xacro:insert_block name="gasket_inertia"/>
       </inertial>
       <visual>
-        <xacro:insert_block name="cylinder_fix" />
+        <xacro:insert_block name="pitch_fix"/>
         <geometry>
-          <cylinder radius="${housing_radius}" length="${gasket_length}" />
+          <cylinder radius="${housing_radius}" length="${gasket_length}"/>
         </geometry>
-        <material name="Orange" />
+        <material name="Orange"/>
       </visual>
       <collision>
-        <xacro:insert_block name="cylinder_fix" />
+        <xacro:insert_block name="pitch_fix"/>
         <geometry>
-          <cylinder radius="${housing_radius}" length="${gasket_length}" />
+          <cylinder radius="${housing_radius}" length="${gasket_length}"/>
         </geometry>
       </collision>
     </link>
   </xacro:macro>
-  <xacro:gasket prefix="fwd" reflect="1" />
-  <xacro:gasket prefix="aft" reflect="-1" />
-  <!--  Dome/Endcap  -->
+  <xacro:gasket prefix="fwd" reflect="1"/>
+  <xacro:gasket prefix="aft" reflect="-1"/>
+  <!--    Dome    -->
   <joint name="dome_joint" type="fixed">
-    <origin xyz="${gasket_length/2} 0 0" rpy="0 0 0" />
-    <parent link="fwd_gasket" />
-    <child link="dome" />
-  </joint>
-  <joint name="endcap_joint" type="fixed">
-    <origin xyz="${-(endcap_length+gasket_length)/2} 0 0" rpy="0 0 0" />
-    <parent link="aft_gasket" />
-    <child link="endcap" />
+    <origin xyz="${gasket_length/2} 0 0" rpy="0 0 0"/>
+    <parent link="fwd_gasket"/>
+    <child link="dome"/>
   </joint>
   <link name="dome">
     <inertial>
-      <mass value="${dome_mass}" />
-      <xacro:insert_block name="dome_inertia" />
+      <mass value="${dome_mass}"/>
+      <xacro:insert_block name="dome_inertia"/>
     </inertial>
     <visual>
       <geometry>
-        <sphere radius="${housing_radius}" />
-        <!-- <mesh filename="package://jaws2_description/meshes/dome.stl" /> -->
+        <sphere radius="${housing_radius}"/>
+        <!-- <mesh filename="package://jaws2_description/meshes/dome.stl"/> -->
       </geometry>
-      <material name="Grey" />
+      <material name="Grey"/>
     </visual>
     <collision>
       <geometry>
-        <sphere radius="${housing_radius}" />
+        <sphere radius="${housing_radius}"/>
       </geometry>
     </collision>
   </link>
+  <!--    Endcap    -->
+  <joint name="endcap_joint" type="fixed">
+    <origin xyz="${-(endcap_length+gasket_length)/2} 0 0" rpy="0 0 0"/>
+    <parent link="aft_gasket"/>
+    <child link="endcap"/>
+  </joint>
   <link name="endcap">
     <inertial>
-      <mass value="${endcap_mass}" />
-      <xacro:insert_block name="endcap_inertia" />
+      <mass value="${endcap_mass}"/>
+      <xacro:insert_block name="endcap_inertia"/>
     </inertial>
     <visual>
-      <xacro:insert_block name="cylinder_fix" />
+      <xacro:insert_block name="pitch_fix"/>
       <geometry>
-        <cylinder radius="${housing_radius}" length="${endcap_length}" />
+        <cylinder radius="${housing_radius}" length="${endcap_length}"/>
       </geometry>
-      <material name="Grey" />
+      <material name="Grey"/>
     </visual>
     <collision>
-      <xacro:insert_block name="cylinder_fix" />
+      <xacro:insert_block name="pitch_fix"/>
       <geometry>
-        <cylinder radius="${housing_radius}" length="${endcap_length}" />
+        <cylinder radius="${housing_radius}" length="${endcap_length}"/>
       </geometry>
     </collision>

File: jaws2_description/urdf/jaws2_mounting.urdf.xacro (robot description, xacro)
@@ -1,29 +1,32 @@
 <?xml version="1.0"?>
 <robot xmlns:xacro="http://ros.org/wiki/xacro">
-  <!--  Port & Starboard Servos  -->
+<!--                     -->
+<!--  Thruster Mounting  -->
+<!--                     -->
+  <!--    Port & Starboard Servos    -->
   <xacro:macro name="servo" params="prefix reflect mirror">
     <joint name="${prefix}_servo" type="revolute">
-      <origin xyz="${shaft_x} ${reflect*shaft_y} 0" rpy="0 ${-M_PI/2} ${mirror}"/>
-      <parent link="housing" />
-      <child link="${prefix}_servo_shaft" />
-      <axis xyz="0 1 0" />
-      <limit lower="${-2*M_PI/3}" upper="${2*M_PI/3}" effort="1.4994" velocity="1.9666" />
+      <origin xyz="${shaft_x} ${reflect*shaft_y} 0" rpy="0 ${zero} ${mirror}"/>
+      <parent link="housing"/>
+      <child link="${prefix}_servo_shaft"/>
+      <axis xyz="${servo_axis}"/>
+      <limit lower="${min}" upper="${max}" effort="${tau}" velocity="${vel}"/>
     </joint>
     <link name="${prefix}_servo_shaft">
       <inertial>
-        <mass value="${shaft_mass}" />
-        <xacro:insert_block name="shaft_inertia" />
+        <mass value="${shaft_mass}"/>
+        <xacro:insert_block name="shaft_inertia"/>
       </inertial>
       <visual>
-        <origin xyz="0 0 0" rpy="${M_PI/2} 0 0" />
+        <xacro:insert_block name="roll_fix"/>
         <geometry>
-          <cylinder radius="${shaft_radius}" length="${shaft_length}" />
+          <cylinder radius="${shaft_radius}" length="${shaft_length}"/>
         </geometry>
-        <material name="DarkGrey" />
+        <material name="DarkGrey"/>
       </visual>
       <collision>
-        <origin xyz="0 0 0" rpy="${M_PI/2} 0 0" />
+        <xacro:insert_block name="roll_fix"/>
         <geometry>
-          <cylinder radius="${shaft_radius}" length="${shaft_length}" />
+          <cylinder radius="${shaft_radius}" length="${shaft_length}"/>
         </geometry>
       </collision>
@@ -32,41 +35,41 @@
   <xacro:servo prefix="port" reflect="1" mirror="0"/>
   <xacro:servo prefix="stbd" reflect="-1" mirror="${M_PI}"/>
-  <!--  Aft Thruster Riser  -->
+  <!--    Aft Thruster Riser    -->
   <joint name="aft_thruster_riser_joint" type="fixed">
-    <origin xyz="${riser_x} 0 ${riser_z}" rpy="0 0 0" />
-    <parent link="housing" />
-    <child link="aft_thruster_riser" />
+    <origin xyz="${riser_x} 0 ${riser_z}" rpy="0 0 0"/>
+    <parent link="housing"/>
+    <child link="aft_thruster_riser"/>
   </joint>
   <link name="aft_thruster_riser">
     <inertial>
-      <mass value="${riser_mass}" />
-      <xacro:insert_block name="riser_inertia" />
+      <mass value="${riser_mass}"/>
+      <xacro:insert_block name="riser_inertia"/>
     </inertial>
     <visual>
       <geometry>
-        <box size="${0.75*riser_length} ${0.55*riser_width} ${riser_height}" />
+        <box size="${0.75*riser_length} ${0.55*riser_width} ${riser_height}"/>
       </geometry>
-      <material name="DarkGrey" />
+      <material name="DarkGrey"/>
     </visual>
     <collision>
       <geometry>
-        <box size="${riser_length} ${riser_width} ${riser_height}" />
+        <box size="${riser_length} ${riser_width} ${riser_height}"/>
       </geometry>
     </collision>
   </link>
-  <!--  Port & Stbd Shaft Seals  -->
+  <!--    Port & Stbd Shaft Seals    -->
   <xacro:macro name="thruster_mounts" params="prefix reflect">
     <joint name="${prefix}_thruster_mount_joint" type="fixed">
       <origin xyz="${shaft_x} ${reflect*(shaft_y-shaft_length)} 0" rpy="0 0 0"/>
-      <parent link="housing" />
-      <child link="${prefix}_thruster_mount" />
+      <parent link="housing"/>
+      <child link="${prefix}_thruster_mount"/>
     </joint>
     <link name="${prefix}_thruster_mount">
       <visual>
-        <origin xyz="0 0 0" rpy="${M_PI/2} 0 0" />
+        <xacro:insert_block name="roll_fix"/>
         <geometry>
-          <cylinder radius="${shaft_radius*0.75}" length="${shaft_length}" />
+          <cylinder radius="${shaft_radius*0.75}" length="${shaft_length}"/>
         </geometry>
-        <material name="FlatBlack" />
+        <material name="FlatBlack"/>
       </visual>
     </link>
@@ -74,16 +77,16 @@
   <xacro:thruster_mounts prefix="port" reflect="1"/>
   <xacro:thruster_mounts prefix="stbd" reflect="-1"/>
-  <!--  Aft Thruster Mounting Point  -->
+  <!--    Aft Thruster Mounting Point    -->
   <joint name="aft_thruster_mount_joint" type="fixed">
-    <origin xyz="${riser_x} 0 ${riser_z-riser_height}" rpy="0 0 0" />
-    <parent link="housing" />
-    <child link="aft_thruster_mount" />
+    <origin xyz="${riser_x} 0 ${riser_z-riser_height}" rpy="0 0 0"/>
+    <parent link="housing"/>
+    <child link="aft_thruster_mount"/>
   </joint>
   <link name="aft_thruster_mount">
     <visual>
       <geometry>
-        <cylinder radius="${riser_length/2}" length="${riser_height}" />
+        <cylinder radius="${riser_length/2}" length="${riser_height}"/>
       </geometry>
-      <material name="FlatBlack" />
+      <material name="FlatBlack"/>
     </visual>
   </link>

File: jaws2_description/urdf/jaws2_properties.urdf.xacro (robot description, xacro)
@@ -1,83 +1,91 @@
 <?xml version="1.0"?>
 <robot xmlns:xacro="http://ros.org/wiki/xacro">
-  <xacro:property name="M_PI" value="3.14159266" />
-  <!--  Housing Properties  -->
-  <xacro:property name="housing_radius" value="0.0762" />
-  <xacro:property name="middle_radius" value="0.06985" />
-  <xacro:property name="fwd_length" value="0.0492" />
-  <xacro:property name="mid_length" value="0.2826" />
-  <xacro:property name="aft_length" value="0.0238" />
-  <xacro:property name="housing_mass" value="1.8914" />
+  <xacro:property name="M_PI" value="3.14159266"/>
+  <xacro:property name="pitch_fix">
+    <origin xyz="0 0 0" rpy="0 ${M_PI/2} 0"/>
+  </xacro:property>
+  <xacro:property name="roll_fix">
+    <origin xyz="0 0 0" rpy="${M_PI/2} 0 0"/>
+  </xacro:property>
+  <xacro:property name="servo_axis" value="0 1 0"/>
+  <xacro:property name="zero" value="${-M_PI/2}"/>
+  <xacro:property name="vel" value="1.96666666"/>
+  <xacro:property name="tau" value="1.49940000"/>
+  <xacro:property name="max" value="${5*M_PI/6}"/>
+  <xacro:property name="min" value="${-5*M_PI/6}"/>
+  <xacro:property name="housing_radius" value="0.0762"/>
+  <xacro:property name="middle_radius" value="0.06985"/>
+  <xacro:property name="fwd_length" value="0.0492"/>
+  <xacro:property name="mid_length" value="0.2826"/>
+  <xacro:property name="aft_length" value="0.0238"/>
+  <xacro:property name="housing_mass" value="1.8914"/>
   <xacro:property name="housing_inertia">
     <inertia ixx="0.00921641" ixy="0.0" ixz="0.0"
              iyy="0.03285281" iyz="0.0"
-             izz="0.03285281" />
+             izz="0.03285281"/>
   </xacro:property>
-  <!-- Gasket Properties  -->
-  <xacro:property name="gasket_length" value="0.0032" />
-  <xacro:property name="gasket_x" value="0.1794" />
-  <xacro:property name="gasket_mass" value="0.0165" />
+  <xacro:property name="gasket_length" value="0.0032"/>
+  <xacro:property name="gasket_x" value="0.1794"/>
+  <xacro:property name="gasket_mass" value="0.0165"/>
   <xacro:property name="gasket_inertia">
     <inertia ixx="0.00004790" ixy="0.0" ixz="0.0"
              iyy="0.00002397" iyz="0.0"
-             izz="0.00002397" />
+             izz="0.00002397"/>
   </xacro:property>
-  <!--  Dome Properties  -->
-  <xacro:property name="dome_mass" value="0.7700" />
+  <xacro:property name="dome_mass" value="0.7700"/>
   <xacro:property name="dome_inertia">
     <inertia ixx="0.003" ixy="0.0" ixz="0.0"
              iyy="0.003" iyz="0.0"
-             izz="0.003" />
+             izz="0.003"/>
   </xacro:property>
-  <!--  Endcap Properties  -->
-  <xacro:property name="endcap_length" value="0.0200" />
-  <xacro:property name="endcap_mass" value="0.1925" />
+  <xacro:property name="endcap_length" value="0.0200"/>
+  <xacro:property name="endcap_mass" value="0.1925"/>
   <xacro:property name="endcap_inertia">
   <inertia ixx="0.000" ixy="0.0" ixz="0.0"
            iyy="0.003" iyz="0.0"
-           izz="0.003" />
+           izz="0.003"/>
   </xacro:property>
-<!--  Port & Stbd Servo Propeties  -->
-  <xacro:property name="shaft_radius" value="0.01580619" />
-  <xacro:property name="shaft_length" value="0.02381250" />
-  <xacro:property name="shaft_x" value="0.14287500" />
-  <xacro:property name="shaft_y" value="0.09763125" />
-  <xacro:property name="shaft_mass" value="0.02320847" />
+  <xacro:property name="servo_axis" value="0 1 0"/>
+  <xacro:property name="zero" value="${-M_PI/2}"/>
+  <xacro:property name="vel" value="1.96666666"/>
+  <xacro:property name="tau" value="1.49940000"/>
+  <xacro:property name="max" value="${5*M_PI/6}"/>
+  <xacro:property name="min" value="${-5*M_PI/6}"/>
+  <xacro:property name="shaft_radius" value="0.01580619"/>
+  <xacro:property name="shaft_length" value="0.02381250"/>
+  <xacro:property name="shaft_x" value="0.14287500"/>
+  <xacro:property name="shaft_y" value="0.09763125"/>
+  <xacro:property name="shaft_mass" value="0.02320847"/>
   <xacro:property name="shaft_inertia">
     <inertia ixx="0.00000444" ixy="0.0" ixz="0.0"
              iyy="0.00000506" iyz="0.0"
-             izz="0.00000444" />
+             izz="0.00000444"/>
   </xacro:property>
-<!--  Aft Thruster Riser Properties  -->
-  <xacro:property name="riser_length" value="0.0260" />
-  <xacro:property name="riser_width" value="0.0260" />
-  <xacro:property name="riser_height" value="0.0127" />
-  <xacro:property name="riser_x" value="-0.13970000" />
-  <xacro:property name="riser_z" value="0.08413750" />
-  <xacro:property name="riser_mass" value="0.02320847" />
+  <xacro:property name="riser_length" value="0.0260"/>
+  <xacro:property name="riser_width" value="0.0260"/>
+  <xacro:property name="riser_height" value="0.0127"/>
+  <xacro:property name="riser_x" value="-0.13970000"/>
+  <xacro:property name="riser_z" value="0.08413750"/>
+  <xacro:property name="riser_mass" value="0.02320847"/>
   <xacro:property name="riser_inertia">
     <inertia ixx="0.00000162" ixy="0.0" ixz="0.0"
              iyy="0.00000162" iyz="0.0"
-             izz="0.00000262" />
+             izz="0.00000262"/>
   </xacro:property>
-  <!--  Miscellaneous  -->
-  <xacro:property name="cylinder_fix">
-    <origin xyz="0 0 0" rpy="0 ${M_PI/2} 0" />
-  </xacro:property>
-    <!--  Rviz Materials  -->
-    <material name="FlatBlack">
-      <color rgba="0.1 0.1 0.1 1.0" />
-    </material>
-    <material name="DarkGrey">
-      <color rgba="0.175 0.175 0.175 1.0" />
-    </material>
-    <material name="Grey">
-      <color rgba="0.3 0.3 0.3 1.0" />
-    </material>
-    <material name="GreyTransparent">
-      <color rgba="0.5 0.5 0.5 0.5" />
-    </material>
-    <material name="Orange">
-      <color rgba="1 0.5088 0.0468 1" />
-    </material>
+  <!--    Rviz Materials    -->
+  <material name="FlatBlack">
+    <color rgba="0.1 0.1 0.1 1.0"/>
+  </material>
+  <material name="DarkGrey">
+    <color rgba="0.175 0.175 0.175 1.0"/>
+  </material>
+  <material name="Grey">
+    <color rgba="0.3 0.3 0.3 1.0"/>
+  </material>
+  <material name="GreyTransparent">
+    <color rgba="0.5 0.5 0.5 0.5"/>
+  </material>
+  <material name="Orange">
+    <color rgba=".75 0.3816 0.0351 1"/>
+  </material>
 </robot>
