Commit message: The great xacro overhault.

File: jaws2_description/urdf/seabotix_properties.urdf.xacro (robot description, xacro)
@@ -1,13 +1,9 @@
 <?xml version="1.0"?>
 <robot xmlns:xacro="http://ros.org/wiki/xacro">
-  <xacro:property name="thruster_mass" value="0.7090" />
-  <xacro:property name="thruster_mass_ctr" value="0 0 0" />
-  <xacro:property name="thruster_volume" value="0.00036933" />
-  <xacro:property name="thruster_vol_ctr" value="0 0 0" />
-  <xacro:property name="body_radius" value="0.02222500" />
-  <xacro:property name="nozzle_radius" value="0.04740000" />
-  <xacro:property name="body_length" value="0.17610000" />
-  <xacro:property name="nozzle_length" value="0.05030000" />
-  <xacro:property name="aft_thruster_x" value="-0.02931250" />
+  <xacro:property name="body_radius" value="0.02222500"/>
+  <xacro:property name="body_length" value="0.17610000"/>
+  <xacro:property name="aft_thruster_x" value="-0.02931250"/>
+  <xacro:property name="thruster_volume" value="0.00036933"/>
+  <xacro:property name="thruster_mass" value="0.70900000"/>
   <xacro:property name="thruster_inertia">
     <inertia ixx="0.00017511" ixy="0.0000" ixz="0.0000"
@@ -15,4 +11,7 @@
              izz="0.00191980"/>
   </xacro:property>
+  <xacro:property name="nozzle_radius" value="0.04740000"/>
+  <xacro:property name="nozzle_length" value="0.05030000"/>
+  <!--  Thruster Materials  -->
   <xacro:macro name="thruster_gazebo" params="prefix">
     <gazebo reference="${prefix}_thruster">
@@ -26,6 +25,6 @@
     </gazebo>
   </xacro:macro>
-  <xacro:thruster_gazebo prefix="port" />
-  <xacro:thruster_gazebo prefix="stbd" />
-  <xacro:thruster_gazebo prefix="aft" />
+  <xacro:thruster_gazebo prefix="port"/>
+  <xacro:thruster_gazebo prefix="stbd"/>
+  <xacro:thruster_gazebo prefix="aft"/>
 </robot>

File: jaws2_description/urdf/seabotix_thrusters.urdf.xacro (robot description, xacro)
@@ -1,24 +1,41 @@
 <?xml version="1.0" ?>
 <robot xmlns:xacro="http://ros.org/wiki/xacro">
-  <!-- http://www.seabotix.com/products/pdf_files/BTD150_Data_Sheet.pdf -->
-  <xacro:include filename="seabotix_properties.urdf.xacro" />
-  <!-- Build the Thrusters -->
+<!--                      -->
+<!--  Seabotix Thrusters  -->
+<!--                      -->
+  <xacro:include filename="seabotix_properties.urdf.xacro"/>
+  <!--    Thruster Joints    -->
+  <xacro:macro name="thruster_joints" params="prefix">
+    <joint name="${prefix}_thruster_joint" type="fixed">
+      <origin xyz="0 ${body_radius+shaft_length/2} 0" rpy="0 0 0"/>
+      <parent link="${prefix}_servo_shaft"/>
+      <child link="${prefix}_thruster"/>
+    </joint>
+  </xacro:macro>
+  <xacro:thruster_joints prefix="port"/>
+  <xacro:thruster_joints prefix="stbd"/>
+  <joint name="aft_thruster_joint" type="fixed">
+    <origin xyz="${aft_thruster_x} 0 ${body_radius+riser_height/2}" rpy="0 0 0"/>
+    <parent link="aft_thruster_riser"/>
+    <child link="aft_thruster"/>
+  </joint>
+  <!--    Thruster Links    -->
   <xacro:macro name="thruster" params="prefix">
     <link name="${prefix}_thruster">
       <inertial>
-        <mass value="${thruster_mass}" />
-        <xacro:insert_block name="thruster_inertia" />
+        <mass value="${thruster_mass}"/>
+        <xacro:insert_block name="thruster_inertia"/>
       </inertial>
       <visual>
-        <xacro:insert_block name="cylinder_fix" />
+        <xacro:insert_block name="pitch_fix"/>
         <geometry>
-          <cylinder radius="${body_radius}" length="${body_length-(2*body_radius)}" />
+          <cylinder radius="${body_radius}" length="${body_length-(2*body_radius)}"/>
         </geometry>
-        <material name="Grey" />
+        <material name="Grey"/>
       </visual>
       <collision>
-        <xacro:insert_block name="cylinder_fix" />
+        <xacro:insert_block name="pitch_fix"/>
         <geometry>
-          <cylinder radius="${body_radius}" length="${body_length}" />
+          <cylinder radius="${body_radius}" length="${body_length}"/>
         </geometry>
       </collision>
@@ -27,46 +44,31 @@
       <visual>
         <geometry>
-          <sphere radius="${body_radius}" />
+          <sphere radius="${body_radius}"/>
         </geometry>
-        <material name="DarkGrey" />
+        <material name="DarkGrey"/>
       </visual>
     </link>
     <link name="${prefix}_thruster_nozzle">
       <visual>
-        <xacro:insert_block name="cylinder_fix" />
+        <xacro:insert_block name="pitch_fix"/>
         <geometry>
-          <cylinder radius="${nozzle_radius}" length="${nozzle_length}" />
+          <cylinder radius="${nozzle_radius}" length="${nozzle_length}"/>
         </geometry>
-        <material name="DarkGrey" />
+        <material name="DarkGrey"/>
       </visual>
     </link>
     <joint name="${prefix}_thruster_nose_cone" type="fixed">
       <origin xyz="${body_length/2-body_radius} 0 0" rpy="0 0 0"/>
-      <parent link="${prefix}_thruster" />
-      <child link="${prefix}_thruster_nose_cone" />
+      <parent link="${prefix}_thruster"/>
+      <child link="${prefix}_thruster_nose_cone"/>
     </joint>
     <joint name="${prefix}_thruster_nozzle" type="fixed">
       <origin xyz="-${(body_length-nozzle_length)/2} 0 0" rpy="0 0 0"/>
-      <parent link="${prefix}_thruster" />
-      <child link="${prefix}_thruster_nozzle" />
+      <parent link="${prefix}_thruster"/>
+      <child link="${prefix}_thruster_nozzle"/>
     </joint>
   </xacro:macro>
-  <xacro:thruster prefix="port" />
-  <xacro:thruster prefix="stbd" />
-  <xacro:thruster prefix="aft" />
-  <!-- Attach the Thrusters -->
-  <xacro:macro name="thruster_joints" params="prefix">
-    <joint name="${prefix}_thruster_joint" type="fixed">
-      <origin xyz="0 ${body_radius+shaft_length/2} 0" rpy="0 0 0"/>
-      <parent link="${prefix}_servo_shaft" />
-      <child link="${prefix}_thruster" />
-    </joint>
-  </xacro:macro>
-  <xacro:thruster_joints prefix="port" />
-  <xacro:thruster_joints prefix="stbd" />
-  <joint name="aft_thruster_joint" type="fixed">
-    <origin xyz="${aft_thruster_x} 0 ${body_radius+riser_height/2}" rpy="0 0 0" />
-    <parent link="aft_thruster_riser" />
-    <child link="aft_thruster" />
-  </joint>
+  <xacro:thruster prefix="port"/>
+  <xacro:thruster prefix="stbd"/>
+  <xacro:thruster prefix="aft"/>
 </robot>

Commit message: Added ballast to prevent Jaws 2 from entering orbit.

File: jaws2_description/urdf/jaws2.gazebo.xacro (robot description, xacro)
@@ -52,4 +52,7 @@
       <material>Gazebo/DarkGrey</material>
     </gazebo>
+    <gazebo reference="${ps}_ballast">
+      <material>Gazebo/DarkGrey</material>
+    </gazebo>
   </xacro:macro>
   <xacro:gazebo_materials fa="fwd" ps="port"/>

File: jaws2_description/urdf/jaws2.urdf (robot description, URDF)
Before this commit: robot jaws2, 24 links, 23 joints
Links:
- added link port_ballast, mass 2.375; collision cylinder length=0.283423881405 radius=0.022225; visual cylinder length=0.283423881405 radius=0.022225
- added link stbd_ballast, mass 2.375; collision cylinder length=0.283423881405 radius=0.022225; visual cylinder length=0.283423881405 radius=0.022225
Joints:
- removed joint housing
- added joint housing_joint: type fixed, parent base_link, child housing
- added joint port_ballast_joint: type fixed, parent base_link, child port_ballast, origin xyz=0.0333375 0.053975 -0.098425 rpy=0 0 0
- added joint stbd_ballast_joint: type fixed, parent base_link, child stbd_ballast, origin xyz=0.0333375 -0.053975 -0.098425 rpy=0 0 0

File: jaws2_description/urdf/jaws2_housing.urdf.xacro (robot description, xacro)
@@ -7,5 +7,5 @@
   <link name="base_link"/>
   <!--    Main Housing Inertia    -->
-  <joint name="housing" type="fixed">
+  <joint name="housing_joint" type="fixed">
     <parent link="base_link"/>
     <child link="housing"/>

File: jaws2_description/urdf/jaws2_mounting.urdf.xacro (robot description, xacro)
@@ -1,4 +1,43 @@
 <?xml version="1.0"?>
 <robot xmlns:xacro="http://ros.org/wiki/xacro">
+<!--                    -->
+<!--  Ballast Mounting  -->
+<!--                    -->
+  <xacro:property name="total" value="4.75"/>
+  <xacro:property name="mass" value="${total/2}"/>
+  <xacro:property name="length" value="${mass/2700/2/(M_PI*body_radius*body_radius)}"/>
+  <xacro:property name="inertia">
+    <inertia ixx="${mass*body_radius^2/2}" ixy="0.0" ixz="0.0"
+             iyy="${mass/12*(3*body_radius*body_radius+length*length)}" iyz="0.0"
+             izz="${mass/12*(3*body_radius*body_radius+length*length)}"/>
+  </xacro:property>
+  <xacro:macro name="ballast" params="prefix reflect">
+    <joint name="${prefix}_ballast_joint" type="fixed">
+      <origin xyz="${1.5*body_radius} ${reflect*(housing_radius-body_radius)} -${housing_radius+body_radius}" rpy="0 0 0"/>
+      <parent link="base_link"/>
+      <child link="${prefix}_ballast"/>
+    </joint>
+    <link name="${prefix}_ballast">
+      <inertial>
+        <mass value="${mass}"/>
+        <xacro:insert_block name="inertia"/>
+      </inertial>
+      <visual>
+        <xacro:insert_block name="pitch_fix"/>
+        <geometry>
+            <cylinder radius="${body_radius}" length="${length}"/>
+        </geometry>
+        <material name="Grey"/>
+      </visual>
+      <collision>
+        <xacro:insert_block name="pitch_fix"/>
+        <geometry>
+            <cylinder radius="${body_radius}" length="${length}"/>
+        </geometry>
+      </collision>
+    </link>
+  </xacro:macro>
+  <xacro:ballast prefix="port" reflect="1"/>
+  <xacro:ballast prefix="stbd" reflect="-1"/>
 <!--                     -->
 <!--  Thruster Mounting  -->

File: jaws2_description/urdf/jaws2_properties.urdf.xacro (robot description, xacro)
@@ -8,10 +8,4 @@
     <origin xyz="0 0 0" rpy="${M_PI/2} 0 0"/>
   </xacro:property>
-  <xacro:property name="servo_axis" value="0 1 0"/>
-  <xacro:property name="zero" value="${-M_PI/2}"/>
-  <xacro:property name="vel" value="1.96666666"/>
-  <xacro:property name="tau" value="1.49940000"/>
-  <xacro:property name="max" value="${5*M_PI/6}"/>
-  <xacro:property name="min" value="${-5*M_PI/6}"/>
   <xacro:property name="housing_radius" value="0.0762"/>
   <xacro:property name="middle_radius" value="0.06985"/>
