Commit message: Built an initial Jaws 2 model for simulation.

File: jaws2_description/urdf/jaws2.urdf (robot description, URDF)
Before this commit: robot jaws2, 14 links, 13 joints
Links:
- removed link aft_base
- removed link aft_body
- removed link aft_dome
- removed link aft_duct
- removed link base_dome
- removed link port_base
- removed link port_body
- removed link port_dome
- removed link port_duct
- removed link stbd_base
- removed link stbd_body
- removed link stbd_dome
- removed link stbd_duct
- added link aft_gasket, mass 0.0165; collision cylinder length=0.0032 radius=0.0762; visual cylinder length=0.0032 radius=0.0762
- added link aft_housing; visual cylinder length=0.0238 radius=0.0762
- added link aft_thruster, mass 0.709; collision cylinder length=0.1761 radius=0.022225; visual cylinder length=0.13165 radius=0.022225
- added link aft_thruster_mount; visual cylinder length=0.0127 radius=0.013
- added link aft_thruster_nose_cone; visual sphere radius=0.022225
- added link aft_thruster_nozzle; visual cylinder length=0.0503 radius=0.0474
- added link aft_thruster_riser, mass 0.02320847; collision box size=0.026 0.026 0.0127; visual box size=0.0195 0.0143 0.0127
- added link dome, mass 0.77; collision sphere radius=0.0762; visual sphere radius=0.0762
- added link endcap, mass 0.1925; collision cylinder length=0.02 radius=0.0762; visual cylinder length=0.02 radius=0.0762
- added link fwd_gasket, mass 0.0165; collision cylinder length=0.0032 radius=0.0762; visual cylinder length=0.0032 radius=0.0762
- added link fwd_housing; visual cylinder length=0.0492 radius=0.0762
- added link mid_housing; visual cylinder length=0.2826 radius=0.06985
- added link port_servo_shaft, mass 0.02320847; collision cylinder length=0.0238125 radius=0.01580619; visual cylinder length=0.0238125 radius=0.01580619
- added link port_thruster, mass 0.709; collision cylinder length=0.1761 radius=0.022225; visual cylinder length=0.13165 radius=0.022225
- added link port_thruster_mount; visual cylinder length=0.0238125 radius=0.0118546425
- added link port_thruster_nose_cone; visual sphere radius=0.022225
- added link port_thruster_nozzle; visual cylinder length=0.0503 radius=0.0474
- added link stbd_servo_shaft, mass 0.02320847; collision cylinder length=0.0238125 radius=0.01580619; visual cylinder length=0.0238125 radius=0.01580619
- added link stbd_thruster, mass 0.709; collision cylinder length=0.1761 radius=0.022225; visual cylinder length=0.13165 radius=0.022225
- added link stbd_thruster_mount; visual cylinder length=0.0238125 radius=0.0118546425
- added link stbd_thruster_nose_cone; visual sphere radius=0.022225
- added link stbd_thruster_nozzle; visual cylinder length=0.0503 radius=0.0474
- link base_link: mass 4.31 -> 1.8914; geometry 
Joints:
- removed joint aft-body
- removed joint aft-dome
- removed joint aft-duct
- removed joint base-aft
- removed joint base-dome
- removed joint port-base
- removed joint port-body
- removed joint port-dome
- removed joint port-duct
- removed joint stbd-base
- removed joint stbd-body
- removed joint stbd-dome
- removed joint stbd-duct
- added joint aft_gasket_joint: type fixed, parent base_link, child aft_gasket, origin xyz=-0.1794 0 0 rpy=0 0 0
- added joint aft_housing_joint: type fixed, parent mid_housing, child aft_housing, origin xyz=-0.1532 0 0 rpy=0 0 0
- added joint aft_thruster_joint: type fixed, parent aft_thruster_riser, child aft_thruster, origin xyz=-0.0293125 0 0.028575 rpy=0 0 0
- added joint aft_thruster_mount_joint: type fixed, parent base_link, child aft_thruster_mount, origin xyz=-0.1397 0 0.0714375 rpy=0 0 0
- added joint aft_thruster_nose_cone: type fixed, parent aft_thruster, child aft_thruster_nose_cone, origin xyz=0.065825 0 0 rpy=0 0 0
- added joint aft_thruster_nozzle: type fixed, parent aft_thruster, child aft_thruster_nozzle, origin xyz=-0.0629 0 0 rpy=0 0 0
- added joint aft_thruster_riser_joint: type fixed, parent base_link, child aft_thruster_riser, origin xyz=-0.1397 0 0.0841375 rpy=0 0 0
- added joint dome_joint: type fixed, parent fwd_gasket, child dome, origin xyz=0.0016 0 0 rpy=0 0 0
- added joint endcap_joint: type fixed, parent aft_gasket, child endcap, origin xyz=-0.0116 0 0 rpy=0 0 0
- added joint fwd_gasket_joint: type fixed, parent base_link, child fwd_gasket, origin xyz=0.1794 0 0 rpy=0 0 0
- added joint fwd_housing_joint: type fixed, parent mid_housing, child fwd_housing, origin xyz=0.1659 0 0 rpy=0 0 0
- added joint mid_housing_joint: type fixed, parent base_link, child mid_housing, origin xyz=-0.0127 0 0 rpy=0 0 0
- added joint port_servo: type revolute, parent base_link, child port_servo_shaft, origin xyz=0.142875 0.09763125 0 rpy=0 2.09439510667 0, axis 0 1 0, limit lower=0 upper=2.61799388333 effort=1.4994 velocity=1.9666
- added joint port_thruster_joint: type fixed, parent port_servo_shaft, child port_thruster, origin xyz=0 0.03413125 0 rpy=0 0 0
- added joint port_thruster_mount_joint: type fixed, parent base_link, child port_thruster_mount, origin xyz=0.142875 0.07381875 0 rpy=0 0 0
- added joint port_thruster_nose_cone: type fixed, parent port_thruster, child port_thruster_nose_cone, origin xyz=0.065825 0 0 rpy=0 0 0
- added joint port_thruster_nozzle: type fixed, parent port_thruster, child port_thruster_nozzle, origin xyz=-0.0629 0 0 rpy=0 0 0
- added joint stbd_servo: type revolute, parent base_link, child stbd_servo_shaft, origin xyz=0.142875 -0.09763125 0 rpy=0 2.09439510667 3.14159266, axis 0 1 0, limit lower=0 upper=2.61799388333 effort=1.4994 velocity=1.9666
- added joint stbd_thruster_joint: type fixed, parent stbd_servo_shaft, child stbd_thruster, origin xyz=0 0.03413125 0 rpy=0 0 0
- added joint stbd_thruster_mount_joint: type fixed, parent base_link, child stbd_thruster_mount, origin xyz=0.142875 -0.07381875 0 rpy=0 0 0
- added joint stbd_thruster_nose_cone: type fixed, parent stbd_thruster, child stbd_thruster_nose_cone, origin xyz=0.065825 0 0 rpy=0 0 0
- added joint stbd_thruster_nozzle: type fixed, parent stbd_thruster, child stbd_thruster_nozzle, origin xyz=-0.0629 0 0 rpy=0 0 0

Commit message: Made Rviz interactive, corrected joint limits.

File: jaws2_description/urdf/jaws2.urdf (robot description, URDF)
Before this commit: robot jaws2, 23 links, 22 joints
Joints:
- joint port_servo: limit lower=0 upper=2.61799388333 effort=1.4994 velocity=1.9666 -> lower=0 upper=5.23598776667 effort=1.4994 velocity=1.9666
- joint stbd_servo: limit lower=0 upper=2.61799388333 effort=1.4994 velocity=1.9666 -> lower=0 upper=5.23598776667 effort=1.4994 velocity=1.9666

File: jaws2_description/urdf/jaws2_housing.urdf.xacro (robot description, xacro)
@@ -83,5 +83,5 @@
       <child link="${prefix}_servo_shaft" />
       <axis xyz="0 1 0" />
-      <limit lower="0" upper="${5*M_PI/6}" effort="1.4994" velocity="1.9666" />
+      <limit lower="0" upper="${5*M_PI/3}" effort="1.4994" velocity="1.9666" />
     </joint>
     <link name="${prefix}_servo_shaft">

Commit message: Added visual collision to housing visuals for buoyancy.

File: jaws2_description/urdf/jaws2.urdf (robot description, URDF)
Before this commit: robot jaws2, 23 links, 22 joints
Links:
- link aft_housing: geometry collision cylinder length=0.0238 radius=0.0762; visual cylinder length=0.0238 radius=0.0762
- link fwd_housing: geometry collision cylinder length=0.0492 radius=0.0762; visual cylinder length=0.0492 radius=0.0762
- link mid_housing: geometry collision cylinder length=0.2826 radius=0.06985; visual cylinder length=0.2826 radius=0.06985

File: jaws2_description/urdf/jaws2_visual.urdf.xacro (robot description, xacro)
@@ -21,4 +21,10 @@
         <material name="FlatBlack" />
       </visual>
+      <collision>
+        <xacro:insert_block name="cylinder_fix" />
+        <geometry>
+          <cylinder radius="${radius}" length="${length}" />
+        </geometry>
+      </collision>
     </link>
   </xacro:macro>

Commit message: Corrected servo properties, testing fake mass.

File: jaws2_description/urdf/jaws2.urdf (robot description, URDF)
Before this commit: robot jaws2, 23 links, 22 joints
Links:
- link base_link: mass 1.8914 -> 5.7914
Joints:
- joint port_servo: limit lower=0 upper=5.23598776667 effort=1.4994 velocity=1.9666 -> lower=-2.09439510667 upper=2.09439510667 effort=1.4994 velocity=1.9666; origin xyz=0.142875 0.09763125 0 rpy=0 2.09439510667 0 -> xyz=0.142875 0.09763125 0 rpy=0 -1.57079633 0
- joint stbd_servo: limit lower=0 upper=5.23598776667 effort=1.4994 velocity=1.9666 -> lower=-2.09439510667 upper=2.09439510667 effort=1.4994 velocity=1.9666; origin xyz=0.142875 -0.09763125 0 rpy=0 2.09439510667 3.14159266 -> xyz=0.142875 -0.09763125 0 rpy=0 -1.57079633 3.14159266

File: jaws2_description/urdf/jaws2_housing.urdf.xacro (robot description, xacro)
@@ -79,9 +79,9 @@
   <xacro:macro name="servo" params="prefix reflect mirror">
     <joint name="${prefix}_servo" type="revolute">
-      <origin xyz="${shaft_x} ${reflect*shaft_y} 0" rpy="0 ${2*M_PI/3} ${mirror}"/>
+      <origin xyz="${shaft_x} ${reflect*shaft_y} 0" rpy="0 ${-M_PI/2} ${mirror}"/>
       <parent link="base_link" />
       <child link="${prefix}_servo_shaft" />
       <axis xyz="0 1 0" />
-      <limit lower="0" upper="${5*M_PI/3}" effort="1.4994" velocity="1.9666" />
+      <limit lower="${-2*M_PI/3}" upper="${2*M_PI/3}" effort="1.4994" velocity="1.9666" />
     </joint>
     <link name="${prefix}_servo_shaft">

File: jaws2_description/urdf/jaws2_properties.urdf.xacro (robot description, xacro)
@@ -31,5 +31,6 @@
   <xacro:property name="mid_length" value="0.2826" />
   <xacro:property name="aft_length" value="0.0238" />
-  <xacro:property name="housing_mass" value="1.8914" />
+  <xacro:property name="housing_mass" value="5.7914" />
+  <!-- Mass: 1.8914 -->
   <xacro:property name="housing_inertia">
     <inertia ixx="0.00921641" ixy="0.0" ixz="0.0"

Commit message: Replaced the dome-sphere with a bonafied super-gigantic-dome.

File: jaws2_description/urdf/jaws2.urdf (robot description, URDF)
Before this commit: robot jaws2, 26 links, 25 joints
Links:
- link dome: geometry collision sphere radius=0.0762; visual mesh filename=package://jaws2_description/meshes/dome.stl

File: jaws2_description/urdf/jaws2_housing.urdf.xacro (robot description, xacro)
@@ -90,6 +90,5 @@
     <visual>
       <geometry>
-        <sphere radius="${housing_radius}"/>
-        <!-- <mesh filename="package://jaws2_description/meshes/dome.stl"/> -->
+        <mesh filename="package://jaws2_description/meshes/dome.stl"/>
       </geometry>
       <material name="Grey"/>
